Commit message: relative path uyumluluğu için değişiklikler

File: src/yoda_cpp_package/urdf/model.urdf (robot description, URDF)
Before this commit: robot yoda_car_model, 5 links, 4 joints
Links:
- link link_1: geometry collision mesh filename=package://yoda_cpp_package/meshes/arackasa2.dae scale=1 1 1; visual box size=0.05 0.05 0.02
- link link_2: geometry collision mesh filename=package://yoda_cpp_package/meshes/lastik.dae scale=1 1 1; visual mesh filename=package://yoda_cpp_package/meshes/lastik.dae scale=1 1 1
- link link_2_clone: geometry collision mesh filename=package://yoda_cpp_package/meshes/lastik.dae scale=1 1 1; visual mesh filename=package://yoda_cpp_package/meshes/lastik.dae scale=1 1 1
- link link_2_clone_1: geometry collision mesh filename=package://yoda_cpp_package/meshes/lastik.dae scale=1 1 1; visual mesh filename=package://yoda_cpp_package/meshes/lastik.dae scale=1 1 1
- link link_2_clone_1_clone: geometry collision mesh filename=package://yoda_cpp_package/meshes/lastik.dae scale=1 1 1; visual mesh filename=package://yoda_cpp_package/meshes/lastik.dae scale=1 1 1
